File: hardware/clock-processing.sch (KiCad schematic (older format))
At the start: 6 parts, among them Q4 2N3904, Q5 2N3906

Commit message: replaced old hardware files with the most recent ones tracking CLAUDE.md AI files used in revising the project
Connections:
- net labels added: +10V
- net labels removed: +12V
- wire segments 13 -> 14
Other:
- note removed: "VV"
Changed lines of the file:
@@
 LIBS:petelib
 LIBS:switches
+LIBS:microchip_pic12mcu
+LIBS:microchip_pic16mcu
+LIBS:microchip_pic18mcu
+LIBS:microchip_pic32mcu
 LIBS:trigger-seq-cache
 EELAYER 25 0
@@
 clock.out
 $Comp
-L GND #PWR39
+L GND #PWR040
 U 1 1 5901A90A
 P 2650 3050
-F 0 "#PWR39" H 2650 2800 50  0001 C CNN
+F 0 "#PWR040" H 2650 2800 50  0001 C CNN
 F 1 "GND" H 2650 2900 50  0000 C CNN
 F 2 "" H 2650 3050 50  0000 C CNN
@@
 $EndComp
 $Comp
-L GND #PWR40
+L GND #PWR041
 U 1 1 5901A931
 P 3050 2900
-F 0 "#PWR40" H 3050 2650 50  0001 C CNN
+F 0 "#PWR041" H 3050 2650 50  0001 C CNN
 F 1 "GND" H 3050 2750 50  0000 C CNN
 F 2 "" H 3050 2900 50  0000 C CNN
@@
 $EndComp
 $Comp
-L GND #PWR42
+L GND #PWR042
 U 1 1 5901DCA5
 P 3450 2750
-F 0 "#PWR42" H 3450 2500 50  0001 C CNN
+F 0 "#PWR042" H 3450 2500 50  0001 C CNN
 F 1 "GND" H 3450 2600 50  0000 C CNN
 F 2 "" H 3450 2750 50  0000 C CNN
 F 3 "" H 3450 2750 50  0000 C CNN
 	1    3450 2750
-	1    0    0    -1
-$EndComp
-$Comp
-L +12V #PWR41
-U 1 1 5901DCA6
-P 3250 1500
-F 0 "#PWR41" H 3250 1350 50  0001 C CNN
-F 1 "+12V" H 3250 1640 50  0000 C CNN
-F 2 "" H 3250 1500 50  0000 C CNN
-F 3 "" H 3250 1500 50  0000 C CNN
-	1    3250 1500
 	1    0    0    -1
 $EndComp
@@
 Wire Wire Line
 	2650 3050 2650 2950
-Text Notes 3550 1450 0    60   ~ 0
-VV
+$Comp
+L +10V #PWR043
+U 1 1 5A97BC3A
+P 3250 1400
+F 0 "#PWR043" H 3250 1250 50  0001 C CNN
+F 1 "+10V" H 3250 1540 50  0000 C CNN
+F 2 "" H 3250 1400 50  0000 C CNN
+F 3 "" H 3250 1400 50  0000 C CNN
+	1    3250 1400
+	1    0    0    -1
+$EndComp
+Wire Wire Line
+	3250 1400 3250 1500
 $EndSCHEMATC
