File: hardware/trigger-seq-front-panel.kicad_pcb (KiCad board)
At the start: 2 copper layers, 91.3 x 128.5 mm, 53 parts

Commit message: updates to correct firmware to use clock in detection; MCLRE=OFF, corrected bit locations for IOC interrupts.  updates to schematics/layout
Other:
- board text added: "v3.4"
- board text removed: "v3.3"
Changed lines of the file:
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@@
     (effects (font (size 1.5 1.5) (thickness 0.3)))
   )
-  (gr_text "v3.3" (at 137.5694 154.1212) (layer "F.SilkS")
+  (gr_text "v3.4" (at 137.5694 154.1212) (layer "F.SilkS")
     (effects (font (size 1.5 1.5) (thickness 0.3)))
   )
