File: hardware/trigger-seq-panel.kicad_pcb (KiCad board)
At the start: 2 copper layers, 89.1 x 104.6 mm, 98 parts, among them J1 OUT1, J2 OUT2, J3 RESET, J4 CLOCK_IN, J5 RUN_STOP, J6 UP_DOWN, J7 CLOCK_OUT, P3 SWITCH_PANEL, P8 JACKS_PANEL, Q6 2N3904, SW1 SW_SPDT, SW10 SW_SPDT, SW11 SW_SPDT, SW12 SW_SPDT, SW13 SW_SPDT, SW14 SW_SPDT, SW15 SW_SPDT, SW16 SW_SPDT, SW17 SW_SPDT, SW18 Run/Stop, SW19 Up/Down, SW2 SW_SPDT, SW20 RESET, SW3 SW_SPDT, SW4 SW_SPDT, SW5 SW_SPDT, SW6 SW_SPDT, SW7 SW_SPDT, SW8 SW_SPDT, SW9 SW_DPDT_x2, U2 TL072

Commit message: updates to correct firmware to use clock in detection; MCLRE=OFF, corrected bit locations for IOC interrupts.  updates to schematics/layout
Parts:
- J4: value CLOCK_IN -> CKIN; footprint My Library:thonkiconn -> myfootprints:thonkiconn_stereo; moved to F.Cu
- P8: footprint Connector_PinSocket_2.54mm:PinSocket_2x07_P2.54mm_Vertical -> Connector_PinSocket_2.54mm:PinSocket_2x08_P2.54mm_Vertical
- turned J4 to 180 degrees
Connections:
- net 2x8/1x16 renamed 2x8/1x16
- net R/S renamed R/S
- net U/D renamed U/D
- J1 pad 2: (no net) -> unconnected-(J1-Pad2)
- J2 pad 2: (no net) -> unconnected-(J2-Pad2)
- J7 pad 2: (no net) -> unconnected-(J7-Pad2)
- SW1 pad 3: (no net) -> unconnected-(SW1-Pad3)
- SW10 pad 3: (no net) -> unconnected-(SW10-Pad3)
- SW11 pad 3: (no net) -> unconnected-(SW11-Pad3)
- SW12 pad 3: (no net) -> unconnected-(SW12-Pad3)
- SW13 pad 3: (no net) -> unconnected-(SW13-Pad3)
- SW14 pad 3: (no net) -> unconnected-(SW14-Pad3)
- SW15 pad 3: (no net) -> unconnected-(SW15-Pad3)
- SW16 pad 3: (no net) -> unconnected-(SW16-Pad3)
- SW17 pad 3: (no net) -> unconnected-(SW17-Pad3)
- SW2 pad 3: (no net) -> unconnected-(SW2-Pad3)
- SW3 pad 3: (no net) -> unconnected-(SW3-Pad3)
- SW4 pad 3: (no net) -> unconnected-(SW4-Pad3)
- SW5 pad 3: (no net) -> unconnected-(SW5-Pad3)
- SW6 pad 3: (no net) -> unconnected-(SW6-Pad3)
- SW7 pad 3: (no net) -> unconnected-(SW7-Pad3)
- SW8 pad 3: (no net) -> unconnected-(SW8-Pad3)
- SW9 pad 6: (no net) -> unconnected-(SW9-Pad6)
Routing:
- net pg: track 0.00 -> 64.5 mm, vias 0 -> 2
- net CKIN: track 78.9 -> 76.9 mm
- net reset: track 71.0 -> 72.4 mm
Other:
- board text added: "The Gator 3.4 panel PCB trigger/gate sequencer (c)2026 Frogleg Synthesis"
- board text removed: "The Gator 3.5 panel PCB trigger/gate sequencer (c)2026 Frogleg Synthesis"
