File: hardware/clock.kicad_sch (KiCad schematic)
At the start: 42 parts, among them J3 RESET, J4 CLOCK_IN, J5 RUN_STOP, J6 UP_DOWN, J7 CLOCK_OUT, P4 JACKS_MAIN, P6 pickit header, P8 JACKS_PANEL, Q6 2N3904, SW18 Run/Stop, SW19 Up/Down, SW20 RESET, SW9 SW_DPDT_x2, U3 PIC16F15345, U4 LM393

Commit message: updates to correct firmware to use clock in detection; MCLRE=OFF, corrected bit locations for IOC interrupts.  updates to schematics/layout
Parts:
- removed J4: CLOCK_IN, My Library:thonkiconn, symbol altconnector:AudioJack2_Ground_Switch
- removed P4: JACKS_MAIN, Connector_PinHeader_2.54mm:PinHeader_2x07_P2.54mm_Vertical, symbol trigger-seq-rescue:Conn_02x07_Odd_Even-Connector
- removed P8: JACKS_PANEL, Connector_PinSocket_2.54mm:PinSocket_2x07_P2.54mm_Vertical, symbol trigger-seq-rescue:Conn_02x07_Odd_Even-Connector
- added J4: CKIN, myfootprints:thonkiconn_stereo, symbol altconnector:AudioJack3_Ground
- added P4: JACKS_MAIN, Connector_PinHeader_2.54mm:PinHeader_2x08_P2.54mm_Vertical, symbol Connector_Generic:Conn_02x08_Odd_Even
- added P8: JACKS_PANEL, Connector_PinSocket_2.54mm:PinSocket_2x08_P2.54mm_Vertical, symbol Connector_Generic:Conn_02x08_Odd_Even
- J3, J5, J6, J7: footprint My Library:thonkiconn -> myfootprints:thonkiconn
- SW18, SW19: footprint My Library:submini_toggle_SPDT_2267079 -> myfootprints:submini_toggle_SPDT_2267079
- SW20: footprint My Library:C&K_round_pushbutton -> myfootprints:C&K_round_pushbutton
- SW9: footprint My Library:submini_toggle_DPDT_wider -> myfootprints:submini_toggle_DPDT_wider
Connections:
- net +12V: now also P4.13 (Pin_13), P8.13 (Pin_13)
- net +5V: now also P4.1 (Pin_1), P8.1 (Pin_1)
- net -12V: now also P4.14 (Pin_14), P8.14 (Pin_14)
- net 2x8/1x16: now also P4.7 (Pin_7), P8.7 (Pin_7)
- net CKIN: now also J4.T, P4.11 (Pin_11), P8.11 (Pin_11)
- net GND: now also J4.S, P4.2 (Pin_2), P8.2 (Pin_2)
- net R/S: now also P4.8 (Pin_8), P8.8 (Pin_8)
- net U/D: now also P4.9 (Pin_9), P8.9 (Pin_9)
- net ckbuf: now also P4.12 (Pin_12), P8.12 (Pin_12)
- net pg: now also J4.R, P4.15 (Pin_15), P8.15 (Pin_15)
- net rate: now also P4.4 (Pin_4), P8.4 (Pin_4)
- net reset: now also P4.10 (Pin_10), P8.10 (Pin_10)
- net steps: now also P4.5 (Pin_5), P8.5 (Pin_5)
- net swing: now also P4.6 (Pin_6), P8.6 (Pin_6)
- net width: now also P4.3 (Pin_3), P8.3 (Pin_3)
- no-connect marks 3 -> 5
Other:
- note added: "A mono plug will short ring to ground taking advantage of this to identify when a clock in plug is present Can use RA3 pin dual use with programming Vpp because Vpp must be 8V or higher to program the chip"
- note added: "using pg pin in normal operation, with a stereo jack, to detect when there is a plug in the clock in"
- note removed: "footprint pads too small can't fit pins through pcb"
- note removed: "need to validate supply values here"

Commit message: updates to schematic properties, nips and tucks
Other:
- note added: "A mono plug will short ring to ground taking advantage of this to identify when a clock in plug is present Can use RA3 pin dual use with programming Vpp because not doing LVP and MCLRE is disabled"
- note removed: "A mono plug will short ring to ground taking advantage of this to identify when a clock in plug is present Can use RA3 pin dual use with programming Vpp because Vpp must be 8V or higher to program the chip"
- company: (none) -> Frogleg Synthesis
- title: (none) -> Gator Trigger Sequencer
Changed lines of the file:
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@@
 (kicad_sch (version 20211123) (generator eeschema)
   (paper "A4")
+  (title_block
+    (title "Gator Trigger Sequencer")
+    (date "2026-09-19")
+    (rev "3.4")
+    (company "Frogleg Synthesis")
+    (comment 1 "includes width, length, rate, swing, 1x16 or 2x8, run/stop, fwd/back, reset")
+    (comment 2 "simple trigger sequencer")
+  )
   (junction (at 77.47 110.49) (diameter 0) (color 0 0 0 0)
   )
@@
     (effects (font (size 1.524 1.524)) (justify left bottom))
   )
-  (text "A mono plug will short ring to ground\ntaking advantage of this to identify when\na clock in plug is present\nCan use RA3 pin dual use with programming Vpp\nbecause Vpp must be 8V or higher to program the chip"
+  (text "A mono plug will short ring to ground\ntaking advantage of this to identify when\na clock in plug is present\nCan use RA3 pin dual use with programming Vpp\nbecause not doing LVP and MCLRE is disabled"
     (at 15.24 55.88 0)
     (effects (font (size 1.524 1.524)) (justify left bottom))
