File: hardware/main.kicad_sch (KiCad schematic)
At the start: 0 parts

Commit message: updates to schematic properties, nips and tucks
Other:
- company: (none) -> Frogleg Synthesis
- title: (none) -> Gator Trigger Sequencer
Changed lines of the file:
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@@
 (kicad_sch (version 20211123) (generator eeschema)
   (paper "A4")
+  (title_block
+    (title "Gator Trigger Sequencer")
+    (date "2026-09-19")
+    (rev "3.4")
+    (company "Frogleg Synthesis")
+    (comment 1 "includes width, length, rate, swing, 1x16 or 2x8, run/stop, fwd/back, reset")
+    (comment 2 "simple trigger sequencer")
+  )
   (wire (pts (xy 166.37 77.47) (xy 181.61 77.47))
     (stroke (width 0) (type default) (color 0 0 0 0))
