File: hardware/outputs.kicad_sch (KiCad schematic)
At the start: 73 parts, among them J1 OUT1, J2 OUT2, P3 SWITCH_PANEL, SW1 SW_SPDT, SW10 SW_SPDT, SW11 SW_SPDT, SW12 SW_SPDT, SW13 SW_SPDT, SW14 SW_SPDT, SW15 SW_SPDT, SW16 SW_SPDT, SW17 SW_SPDT, SW2 SW_SPDT, SW3 SW_SPDT, SW4 SW_SPDT, SW5 SW_SPDT, SW6 SW_SPDT, SW7 SW_SPDT, SW8 SW_SPDT, SW9 SW_DPDT_x2, U2 TL072

Commit message: updates to correct firmware to use clock in detection; MCLRE=OFF, corrected bit locations for IOC interrupts.  updates to schematics/layout
Parts:
- D10, D19, D20, D21, D22, D23, D24, D25, D26, D3, D4, D5, D6, D7, D8, D9: footprint My Library:LED_D3.0mm -> myfootprints:LED_D3.0mm
- J1, J2: footprint My Library:thonkiconn -> myfootprints:thonkiconn
- SW1, SW10, SW11, SW12, SW13, SW14, SW15, SW16, SW17, SW2, SW3, SW4, SW5, SW6, SW7, SW8: footprint My Library:submini_toggle_SPDT_2267079 -> myfootprints:submini_toggle_SPDT_2267079
- SW9: footprint My Library:submini_toggle_DPDT_wider -> myfootprints:submini_toggle_DPDT_wider

Commit message: updates to schematic properties, nips and tucks
Other:
- company: (none) -> Frogleg Synthesis
- title: (none) -> Gator Trigger Sequencer
Changed lines of the file:
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@@
 (kicad_sch (version 20211123) (generator eeschema)
   (paper "A4")
+  (title_block
+    (title "Gator Trigger Sequencer")
+    (date "2026-09-19")
+    (rev "3.4")
+    (company "Frogleg Synthesis")
+    (comment 1 "includes width, length, rate, swing, 1x16 or 2x8, run/stop, fwd/back, reset")
+    (comment 2 "simple trigger sequencer")
+  )
   (junction (at 43.18 106.68) (diameter 0) (color 0 0 0 0)
   )
