File: hardware/switching.kicad_sch (KiCad schematic)
At the start: 19 parts, among them P7 SWITCH_MAIN, Q1 2N3904, Q2 2N3904, Q3 2N3904, Q4 2N3904, Q5 2N3904, U5 4051, U6 4051, U8 TL072

Commit message: updates to schematic properties, nips and tucks
Other:
- company: (none) -> Frogleg Synthesis
- title: (none) -> Gator Trigger Sequencer
Changed lines of the file:
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@@
 (kicad_sch (version 20211123) (generator eeschema)
   (paper "A4")
+  (title_block
+    (title "Gator Trigger Sequencer")
+    (date "2026-09-19")
+    (rev "3.4")
+    (company "Frogleg Synthesis")
+    (comment 1 "includes width, length, rate, swing, 1x16 or 2x8, run/stop, fwd/back, reset")
+    (comment 2 "simple trigger sequencer")
+  )
   (junction (at 101.6 93.98) (diameter 0) (color 0 0 0 0)
   )
