File: hardware/trigger-seq.kicad_sch (KiCad schematic)
At the start: 0 parts

Commit message: updates to schematic properties, nips and tucks
Other:
- title: Trigger Sequencer -> Gator Trigger Sequencer
Changed lines of the file:
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@@
   (paper "A4")
   (title_block
-    (title "Trigger Sequencer")
+    (title "Gator Trigger Sequencer")
+    (date "2026-09-19")
+    (rev "3.4")
     (company "Frogleg Synthesis")
-    (comment 1 "simple trigger sequencer to go with the 808 boards")
+    (comment 1 "includes width, length, rate, swing, 1x16 or 2x8, run/stop, fwd/back, reset")
+    (comment 2 "simple trigger sequencer")
   )
   (sheet (at 34.29 27.94) (size 45.72 87.63) (fields_autoplaced)
